File: AudioCodec.kicad_sch (KiCad schematic)
At the start: 51 parts, among them U2 ES8388, U3 MP1720

Commit message: add dnp on pull up resistors
Parts:
- R10, R11: now not fitted
Changed lines of the file:
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@@
 		(in_bom yes)
 		(on_board yes)
-		(dnp no)
+		(dnp yes)
 		(property "Reference" "R11"
 			(at 29.718 35.814 90)
@@
 		(in_bom yes)
 		(on_board yes)
-		(dnp no)
+		(dnp yes)
 		(property "Reference" "R10"
 			(at 34.798 35.814 90)
